Commit message: update

File: chapter6/chapter6_ws/install/fishbot_description/share/fishbot_description/urdf/fishbot/base.urdf.xacro (robot description, xacro)
@@ -2,4 +2,5 @@
 <robot xmlns:xacro="http://www.ros.org/wiki/xacro">
   <xacro:macro name="base_xacro" params="length radius">
+    <link name="base_footprint"/>
     <!-- 机器人身体部分 -->
     <link name="base_link">
@@ -18,4 +19,9 @@
         </visual>
     </link>
+    <joint name="joint_name" type="fixed">
+      <origin xyz="0.0 0.0 ${length/2.0+0.032-0.001}" rpy="0.0 0.0 0.0"/>
+      <parent link="base_footprint"/>
+      <child link="base_link"/>
+    </joint>
   </xacro:macro>
 </robot>
