Commit message: update

File: chapter6/chapter6_ws/install/fishbot_description/share/fishbot_description/urdf/fishbot/actuator/caster.urdf.xacro (robot description, xacro)
@@ -6,16 +6,29 @@
         <!-- 部件的外观描述 -->
         <visual>
-        <!-- 沿着自己几何中心的偏移和旋转量 -->
-        <!-- 旋绕自身x轴旋转180度 -->
-        <origin xyz="0.0 0.0 0.0" rpy="0.0 0.0 0.0" />
-        <!-- 几何形状 -->
-        <geometry>
-            <sphere radius="0.016"/>
-        </geometry>
-        <!-- 材质颜色 -->
-        <material name="yellow">
-            <color rgba="1.0 1.0 0.0 0.8"/>
-        </material>
+            <!-- 沿着自己几何中心的偏移和旋转量 -->
+            <!-- 旋绕自身x轴旋转180度 -->
+            <origin xyz="0.0 0.0 0.0" rpy="0.0 0.0 0.0" />
+            <!-- 几何形状 -->
+            <geometry>
+                <sphere radius="0.016"/>
+            </geometry>
+            <!-- 材质颜色 -->
+            <material name="yellow">
+                <color rgba="1.0 1.0 0.0 0.8"/>
+            </material>
         </visual>
+        <collision>
+            <!-- 沿着自己几何中心的偏移和旋转量 -->
+            <!-- 旋绕自身x轴旋转180度 -->
+            <origin xyz="0.0 0.0 0.0" rpy="0.0 0.0 0.0" />
+            <!-- 几何形状 -->
+            <geometry>
+                <sphere radius="0.016"/>
+            </geometry>
+            <!-- 材质颜色 -->
+            <material name="yellow">
+                <color rgba="1.0 1.0 0.0 0.8"/>
+            </material>
+        </collision>
     </link>
     <!-- 机器人的关节, 用于组合机器人的部件 -->

File: chapter6/chapter6_ws/install/fishbot_description/share/fishbot_description/urdf/fishbot/actuator/wheel.urdf.xacro (robot description, xacro)
@@ -6,16 +6,29 @@
         <!-- 部件的外观描述 -->
         <visual>
-        <!-- 沿着自己几何中心的偏移和旋转量 -->
-        <!-- 旋绕自身x轴旋转180度 -->
-        <origin xyz="0.0 0.0 0.0" rpy="1.57079 0.0 0.0" />
-        <!-- 几何形状 -->
-        <geometry>
-            <cylinder radius="0.032" length="0.04"/>
-        </geometry>
-        <!-- 材质颜色 -->
-        <material name="yellow">
-            <color rgba="1.0 1.0 0.0 0.8"/>
-        </material>
+            <!-- 沿着自己几何中心的偏移和旋转量 -->
+            <!-- 旋绕自身x轴旋转180度 -->
+            <origin xyz="0.0 0.0 0.0" rpy="1.57079 0.0 0.0" />
+            <!-- 几何形状 -->
+            <geometry>
+                <cylinder radius="0.032" length="0.04"/>
+            </geometry>
+            <!-- 材质颜色 -->
+            <material name="yellow">
+                <color rgba="1.0 1.0 0.0 0.8"/>
+            </material>
         </visual>
+        <collision>
+            <!-- 沿着自己几何中心的偏移和旋转量 -->
+            <!-- 旋绕自身x轴旋转180度 -->
+            <origin xyz="0.0 0.0 0.0" rpy="1.57079 0.0 0.0" />
+            <!-- 几何形状 -->
+            <geometry>
+                <cylinder radius="0.032" length="0.04"/>
+            </geometry>
+            <!-- 材质颜色 -->
+            <material name="yellow">
+                <color rgba="1.0 1.0 0.0 0.8"/>
+            </material>
+        </collision>
     </link>
     <!-- 机器人的关节, 用于组合机器人的部件 -->

File: chapter6/chapter6_ws/install/fishbot_description/share/fishbot_description/urdf/fishbot/base.urdf.xacro (robot description, xacro)
@@ -7,15 +7,27 @@
         <!-- 部件的外观描述 -->
         <visual>
-        <!-- 沿着自己几何中心的偏移和旋转量 -->
-        <origin xyz="0.0 0.0 0.0" rpy="0.0 0.0 0.0" />
-        <!-- 几何形状 -->
-        <geometry>
-            <cylinder length="${length}" radius="${radius}"/>
-        </geometry>
-        <!-- 材质颜色 -->
-        <material name="white">
-            <color rgba="1.0 1.0 1.0 0.5"/>
-        </material>
+          <!-- 沿着自己几何中心的偏移和旋转量 -->
+          <origin xyz="0.0 0.0 0.0" rpy="0.0 0.0 0.0" />
+          <!-- 几何形状 -->
+          <geometry>
+              <cylinder length="${length}" radius="${radius}"/>
+          </geometry>
+          <!-- 材质颜色 -->
+          <material name="white">
+              <color rgba="1.0 1.0 1.0 0.5"/>
+          </material>
         </visual>
+        <collision>
+          <!-- 沿着自己几何中心的偏移和旋转量 -->
+          <origin xyz="0.0 0.0 0.0" rpy="0.0 0.0 0.0" />
+          <!-- 几何形状 -->
+          <geometry>
+              <cylinder length="${length}" radius="${radius}"/>
+          </geometry>
+          <!-- 材质颜色 -->
+          <material name="white">
+              <color rgba="1.0 1.0 1.0 0.5"/>
+          </material>
+        </collision>
     </link>
     <joint name="joint_name" type="fixed">

File: chapter6/chapter6_ws/install/fishbot_description/share/fishbot_description/urdf/fishbot/sensor/camera.urdf.xacro (robot description, xacro)
@@ -5,15 +5,27 @@
         <!-- 部件的外观描述 -->
         <visual>
-        <!-- 沿着自己几何中心的偏移和旋转量 -->
-        <origin xyz="0.0 0.0 0.0" rpy="0.0 0.0 0.0" />
-        <!-- 几何形状 -->
-        <geometry>
-            <box size="0.02 0.10 0.02"/>
-        </geometry>
-        <!-- 材质颜色 -->
-        <material name="black">
-            <color rgba="0.0 0.0 0.0 0.5"/>
-        </material>
+            <!-- 沿着自己几何中心的偏移和旋转量 -->
+            <origin xyz="0.0 0.0 0.0" rpy="0.0 0.0 0.0" />
+            <!-- 几何形状 -->
+            <geometry>
+                <box size="0.02 0.10 0.02"/>
+            </geometry>
+            <!-- 材质颜色 -->
+            <material name="black">
+                <color rgba="0.0 0.0 0.0 0.5"/>
+            </material>
         </visual>
+        <collision>
+            <!-- 沿着自己几何中心的偏移和旋转量 -->
+            <origin xyz="0.0 0.0 0.0" rpy="0.0 0.0 0.0" />
+            <!-- 几何形状 -->
+            <geometry>
+                <box size="0.02 0.10 0.02"/>
+            </geometry>
+            <!-- 材质颜色 -->
+            <material name="black">
+                <color rgba="0.0 0.0 0.0 0.5"/>
+            </material>
+        </collision>
     </link>
     <!-- 机器人的关节, 用于组合机器人的部件 -->

File: chapter6/chapter6_ws/install/fishbot_description/share/fishbot_description/urdf/fishbot/sensor/imu.urdf.xacro (robot description, xacro)
@@ -6,15 +6,27 @@
         <!-- 部件的外观描述 -->
         <visual>
-        <!-- 沿着自己几何中心的偏移和旋转量 -->
-        <origin xyz="0.0 0.0 0.0" rpy="0.0 0.0 0.0" />
-        <!-- 几何形状 -->
-        <geometry>
-            <box size="0.02 0.02 0.02"/>
-        </geometry>
-        <!-- 材质颜色 -->
-        <material name="black">
-            <color rgba="0.0 0.0 0.0 0.5"/>
-        </material>
+            <!-- 沿着自己几何中心的偏移和旋转量 -->
+            <origin xyz="0.0 0.0 0.0" rpy="0.0 0.0 0.0" />
+            <!-- 几何形状 -->
+            <geometry>
+                <box size="0.02 0.02 0.02"/>
+            </geometry>
+            <!-- 材质颜色 -->
+            <material name="black">
+                <color rgba="0.0 0.0 0.0 0.5"/>
+            </material>
         </visual>
+        <collision>
+            <!-- 沿着自己几何中心的偏移和旋转量 -->
+            <origin xyz="0.0 0.0 0.0" rpy="0.0 0.0 0.0" />
+            <!-- 几何形状 -->
+            <geometry>
+                <box size="0.02 0.02 0.02"/>
+            </geometry>
+            <!-- 材质颜色 -->
+            <material name="black">
+                <color rgba="0.0 0.0 0.0 0.5"/>
+            </material>
+        </collision>
     </link>
     <!-- 机器人的关节, 用于组合机器人的部件 -->

File: chapter6/chapter6_ws/install/fishbot_description/share/fishbot_description/urdf/fishbot/sensor/laser.urdf.xacro (robot description, xacro)
@@ -6,15 +6,27 @@
         <!-- 部件的外观描述 -->
         <visual>
-        <!-- 沿着自己几何中心的偏移和旋转量 -->
-        <origin xyz="0.0 0.0 0.0" rpy="0.0 0.0 0.0" />
-        <!-- 几何形状 -->
-        <geometry>
-            <cylinder radius="0.01" length="0.10"/>
-        </geometry>
-        <!-- 材质颜色 -->
-        <material name="black">
-            <color rgba="0.0 0.0 0.0 1.0"/>
-        </material>
+            <!-- 沿着自己几何中心的偏移和旋转量 -->
+            <origin xyz="0.0 0.0 0.0" rpy="0.0 0.0 0.0" />
+            <!-- 几何形状 -->
+            <geometry>
+                <cylinder radius="0.01" length="0.10"/>
+            </geometry>
+            <!-- 材质颜色 -->
+            <material name="black">
+                <color rgba="0.0 0.0 0.0 1.0"/>
+            </material>
         </visual>
+        <collision>
+            <!-- 沿着自己几何中心的偏移和旋转量 -->
+            <origin xyz="0.0 0.0 0.0" rpy="0.0 0.0 0.0" />
+            <!-- 几何形状 -->
+            <geometry>
+                <cylinder radius="0.01" length="0.10"/>
+            </geometry>
+            <!-- 材质颜色 -->
+            <material name="black">
+                <color rgba="0.0 0.0 0.0 1.0"/>
+            </material>
+        </collision>
     </link>
     <!-- 雷达 -->
@@ -22,15 +34,27 @@
         <!-- 部件的外观描述 -->
         <visual>
-        <!-- 沿着自己几何中心的偏移和旋转量 -->
-        <origin xyz="0.0 0.0 0.0" rpy="0.0 0.0 0.0" />
-        <!-- 几何形状 -->
-        <geometry>
-            <cylinder radius="0.02" length="0.02"/>
-        </geometry>
-        <!-- 材质颜色 -->
-        <material name="black">
-            <color rgba="0.0 0.0 0.0 1.0"/>
-        </material>
+            <!-- 沿着自己几何中心的偏移和旋转量 -->
+            <origin xyz="0.0 0.0 0.0" rpy="0.0 0.0 0.0" />
+            <!-- 几何形状 -->
+            <geometry>
+                <cylinder radius="0.02" length="0.02"/>
+            </geometry>
+            <!-- 材质颜色 -->
+            <material name="black">
+                <color rgba="0.0 0.0 0.0 1.0"/>
+            </material>
         </visual>
+        <collision>
+            <!-- 沿着自己几何中心的偏移和旋转量 -->
+            <origin xyz="0.0 0.0 0.0" rpy="0.0 0.0 0.0" />
+            <!-- 几何形状 -->
+            <geometry>
+                <cylinder radius="0.02" length="0.02"/>
+            </geometry>
+            <!-- 材质颜色 -->
+            <material name="black">
+                <color rgba="0.0 0.0 0.0 1.0"/>
+            </material>
+        </collision>
     </link>
     <!-- 机器人的关节, 用于组合机器人的部件 -->
