Commit message: update

File: chapter6/chapter6_ws/src/fishbot_description/urdf/fishbot/actuator/caster.urdf.xacro (robot description, xacro)
@@ -40,4 +40,10 @@
         <child link="${caster_name}_link"/>
     </joint>
+    <gazebo reference="${caster_name}_link">
+        <mu1 value="0.0"/>
+        <mu2 value="0.0"/>
+        <kp value="1000000000.0"/>
+        <kd value="1.0"/>
+    </gazebo>
   </xacro:macro>
 </robot>

File: chapter6/chapter6_ws/src/fishbot_description/urdf/fishbot/actuator/wheel.urdf.xacro (robot description, xacro)
@@ -43,4 +43,10 @@
         <axis xyz="0 1 0"/>
     </joint>
+    <gazebo reference="${wheel_name}_link">
+        <mu1 value="20.0"/>
+        <mu2 value="20.0"/>
+        <kp value="1000000000.0"/>
+        <kd value="1.0"/>
+    </gazebo>
   </xacro:macro>
 </robot>

File: chapter6/chapter6_ws/src/fishbot_description/urdf/fishbot/sensor/laser.urdf.xacro (robot description, xacro)
@@ -72,4 +72,10 @@
         <child link="laser_cylinder_link"/>
     </joint>
+    <gazebo reference="laser_cylinder_link">
+        <material>Gazebo/Black</material>
+    </gazebo>
+    <gazebo reference="laser_link">
+        <material>Gazebo/Black</material>
+    </gazebo>
   </xacro:macro>
 </robot>
