Commit message: 深度相机仿真

File: chapter6/chapter6_ws/src/fishbot_description/urdf/fishbot/plugins/gazebo_sensor_plugin.xacro (robot description, xacro)
@@ -113,4 +113,29 @@
             </sensor>
         </gazebo>
+        <gazebo reference="camera_link">
+            <sensor type="depth" name="camera_sensor">
+                <plugin name="depth_camera" filename="libgazebo_ros_camera.so">
+                    <frame_name>camera_optical_link</frame_name>
+                </plugin>
+                <always_on>true</always_on>
+                <update_rate>10</update_rate>
+                <camera name="camera">
+                    <horizontal_fov>1.5009831567</horizontal_fov>
+                    <image>
+                        <width>800</width>
+                        <height>600</height>
+                        <format>R8G8B8</format>
+                    </image>
+                    <distortion>
+                        <k1>0.0</k1>
+                        <k2>0.0</k2>
+                        <k3>0.0</k3>
+                        <p1>0.0</p1>
+                        <p2>0.0</p2>
+                        <center>0.5 0.5</center>
+                    </distortion>
+                </camera>
+            </sensor>
+        </gazebo>
     </xacro:macro>
 </robot>

File: chapter6/chapter6_ws/src/fishbot_description/urdf/fishbot/sensor/camera.urdf.xacro (robot description, xacro)
@@ -31,4 +31,11 @@
         <xacro:box_inertia m="0.1" w="0.02" h="0.10" d="0.02"/>
     </link>
+    <link name="camera_optical_link"></link>
+    <!-- 机器人的关节, 用于组合机器人的部件 -->
+    <joint name="camera_optical_joint" type="fixed">
+        <origin xyz="${xyz}" rpy="${-pi/2} 0.0 ${-pi/2}"/>
+        <parent link="camera_link"/>
+        <child link="camera_optical_link"/>
+    </joint>
     <!-- 机器人的关节, 用于组合机器人的部件 -->
     <joint name="camera_joint" type="fixed">
